File: Hardware/Alligator_Components PSRAM 100pin.sch (KiCad schematic (older format))
At the start: 79 parts, among them J1 SWD_Header, J2 Eurorack_10_pin_power, J3 Conn_01x20_Female, U1 STM32H743ZITx, U2 IS42S16400J-xC, U3 MCP6004, U4 PCM5100APW, U5 TL072, U7 LM1117-3.3, Y1 8MHz 20pF

Commit message: Updates to schematic; Output ADC data over I2S via interrupt with L/R awareness
Parts:
- removed J3: Conn_01x20_Female, symbol Connector:Conn_01x20_Female
- added C? (x2): 2.2uF, symbol Device:C_Small
- added C? (x2): 30pF, symbol Device:C_Small
- added C? (x6): 100nF, symbol Device:C_Small
- added U?: STM32H743VITx, Package_QFP:LQFP-100_14x14mm_P0.5mm, symbol MCU_ST_STM32H7:STM32H743VITx
- added Y1: 8MHz 20pF, Crystals:Crystal_SMD_0603-2pin_6.0x3.5mm_HandSoldering, symbol Device:Crystal
- R13: value 6k8 -> 47k
- R8: value 20k -> 68k
- R9: value 47k -> 100k
- renumbered C6 to C?, C4 to C?, C2 to C?, C3 to C?, C5 to C?, C7 to C?, C8 to C?, C9 to C?, C10 to C?, C11 to C?, C14 to C?, C15 to C?, C19 to C?, C21 to C?, C1 to C?, C12 to C?, C44 to C?, C20 to C?, C25 to C?, C26 to C?, C37 to C?, C42 to C?, C16 to C?, J2 to J?, U2 to U?, U1 to U?, Y1 to Y?
Connections:
- net labels added: HARM1_CVIN, HARM2_CVIN, PITCH_CVIN, WARP_CVIN
- net labels removed: ADC123_INP11, ADC12_INP14, ADC12_INP15, ADC12_INP18, ADC12_INP19, ADC12_INP3, ADC12_INP4, ADC12_INP5, ADC12_INP7, ADC12_INP8, ADC12_INP9, ADC1_INP16, ADC1_INP17, CV_IN1, CV_IN2, CV_IN3, CV_IN4
- wire segments 413 -> 435
- no-connect marks 56 -> 2
Other:
- moved on the sheet: C?, J1, U?, Y?
