File: Hardware/Alligator_Components.sch (KiCad schematic (older format))
At the start: 118 parts, among them J1 SWD_Header, J2 Eurorack_10_pin_power, J3 Conn_01x20_Female, U1 STM32H743ZITx, U2 IS42S16400J-xC, U3 PCM5100APW, U4 SSI2164, U5 MCP6004, U6 MCP6004, U7 TL074, U8 LM1117-3.3, Y1 8MHz 20pF

Commit message: First Draft of Component Schematic Done; Added enum for ADC input selction
Parts:
- removed C?: 1.5nF, symbol Device:C_Small
- removed J3: Conn_01x20_Female, symbol Connector:Conn_01x20_Female
- removed R?: 56k, Resistors_SMD:R_0805_HandSoldering, symbol Device:R
- removed R?: 91k, Resistors_SMD:R_0805_HandSoldering, symbol Device:R
- removed R?: 100k, Resistors_SMD:R_0805_HandSoldering, symbol Device:R
- removed SW?: SW_Push, symbol Switch:SW_Push
- removed U6: MCP6004, SMD_Packages:SOIC-14_N, symbol Amplifier_Operational:MCP6004
- added J3, J4, J5, J6: Conn_01x08_Female, Socket_Strips:Socket_Strip_Straight_1x08_Pitch2.54mm, symbol Connector:Conn_01x08_Female
- added unit 4 of U6
- C1, C10, C11, C12, C14, C15, C16, C19, C2, C20, C21, C25, C26, C3, C37, C42, C44, C5, C7, C8, C9: footprint (none) -> Capacitors_SMD:C_0603_HandSoldering
- C13, C17, C24, C38: footprint Capacitors_SMD:C_0805_HandSoldering -> Capacitors_SMD:C_0603_HandSoldering
- C18, C23, C27, C28, C29, C30, C32, C34, C45: renamed from C?; footprint (none) -> Capacitors_SMD:C_0603_HandSoldering
- C22, C31, C33, C43: footprint Capacitors_SMD:C_0805_HandSoldering -> Capacitors_SMD:C_0805
- C4, C6: footprint (none) -> Capacitors_SMD:C_0805
- C47, C48, C49, C50, C51, C52: renamed from C?; footprint (none) -> Capacitors_SMD:C_0805
- R1, R10, R14, R2: renamed from R?; footprint (none) -> Resistors_SMD:R_0603_HandSoldering
- R11, R12, R13, R18, R19, R20, R21, R22, R4, R5, R6, R7, R8, R9: footprint Resistors_SMD:R_0805_HandSoldering -> Resistors_SMD:R_0603_HandSoldering
- R15, R16, R17, R3: renamed from R?; value 500R -> 510R; footprint (none) -> Resistors_SMD:R_0603_HandSoldering
- R23, R24, R25, R26, R27, R28, R29, R30, R31, R34, R36, R37, R38, R39, R40, R41, R42, R43: renamed from R?; footprint Resistors_SMD:R_0805_HandSoldering -> Resistors_SMD:R_0603_HandSoldering
- RV1: renamed from RV?; footprint (none) -> Resistors_SMD:R_0603_HandSoldering
- SW1, SW2: renamed from SW?; footprint (none) -> Resistors_SMD:R_0603_HandSoldering
- U7: footprint (none) -> SMD_Packages:SOIC-14_N
- U7: renamed from U?; footprint (none) -> SMD_Packages:SOIC-14_N
Connections:
- net ADC123_INP11 is gone; now on net EXT_AUDIO_IN_R: U1.27 (PC1)
- net ADC12_INP15 is gone; now on net DELAY_CV_SCALED_L: U1.37 (PA3)
- net ADC12_INP3 is gone; now on net EXT_AUDIO_IN_L: U1.42 (PA6)
- net ADC12_INP4 is gone; now on net DELAY_CV_L: U1.44 (PC4)
- net ADC12_INP8 is gone; now on net DELAY_POT_L: U1.45 (PC5)
- net ADC1_INP16 is gone; now on net DELAY_CV_R: U1.34 (PA0)
- net ADC1_INP17 is gone; now on net DELAY_POT_R: U1.35 (PA1)
- net +3.3VA: now also J3.8 (Pin_8), J4.8 (Pin_8), J5.8 (Pin_8), J6.8 (Pin_8), U6.12 (+)
- net CLOCK: now also U6.10 (+), J4.6 (Pin_6); no longer U6.5 (+)
- net CLOCK_SCALED: now also U6.8, U6.9 (-); no longer U6.6 (-), U6.7
- net DELAY_CV_L: now also J5.1 (Pin_1)
- net DELAY_CV_R: now also J5.3 (Pin_3)
- net DELAY_POT_L: now also J5.2 (Pin_2)
- net DELAY_POT_R: now also J5.4 (Pin_4)
- net DRY_OUT_L: now also U7.9 (-); no longer U7.2 (-)
- net DRY_OUT_R: now also U7.13 (-); no longer U7.6 (-)
- net EXT_AUDIO_IN_L: now also J4.1 (Pin_1)
- net EXT_AUDIO_IN_R: now also J4.2 (Pin_2)
- net EXT_AUDIO_OUT_L: now also J4.4 (Pin_4)
- net EXT_AUDIO_OUT_R: now also J4.5 (Pin_5)
- net FEEDBACK_CV: now also J6.3 (Pin_3)
- net FEEDBACK_POT: now also J6.4 (Pin_4)
- net GND: now also U7.10 (+), U7.12 (+), U7.3 (+), U7.5 (+), J3.7 (Pin_7), J4.7 (Pin_7), J5.7 (Pin_7), J6.7 (Pin_7); no longer U7.10 (+), U7.12 (+), U7.3 (+), U7.5 (+)
- net LED1: now also J6.5 (Pin_5)
- net LED2: now also J6.6 (Pin_6)
- net MIX_CV: now also J6.2 (Pin_2)
- net MIX_POT: now also J6.1 (Pin_1)
- net MODE1: now also J3.2 (Pin_2)
- net MODE2: now also J3.3 (Pin_3)
- net RESET: now also J4.3 (Pin_3)
- net at C51.1, R18.1, R20.2: now also U7.8; no longer U7.1
- net at C52.1, R19.1, R21.2: now also U7.14; no longer U7.7
- net USB_VBUS: now reaches U1.101 (PA9)
- net USB_VBUS: now also J3.4 (Pin_4)
- net USB_DM: now reaches U1.103 (PA11)
- net USB_DM: now also J3.5 (Pin_5)
- net USB_DP: now reaches U1.104 (PA12)
- net USB_DP: now also J3.6 (Pin_6)
- net at C49.1, R40.1, R42.2: now also U7.1; no longer U7.8
- net at C49.2, R38.1, R40.2: now also U7.2 (-); no longer U7.9 (-)
- net at C50.2, R39.1, R41.2: now also U7.6 (-); no longer U7.13 (-)
- net at C50.1, R41.1, R43.2: now also U7.7; no longer U7.14
- net DELAY_CHORUS: now reaches SW1.2 (B)
- net DELAY_CHORUS: now also J3.1 (Pin_1)
- net MIX_DRY renamed MIX_DRY_CTL
- net MIX_WET renamed MIX_WET_CTL
- new net: U6.13 (-), U6.14
- new net ADC12_INP14_PA2_IN: J5.6 (Pin_6)
- new net ADC12_INP7_PA7_IN: J5.5 (Pin_5)
- no-connect marks 59 -> 71
Other:
- note added: "DAC and VCAs"
- note added: "DRAM"
- note added: "Delay: Dual Mono, Ping Ping\nChorus: Chorus/Flange (w feedback?)"
- note added: "Headers and Connectors"
- note added: "Input Scaling"
- note added: "Microcontroller"
- note added: "Output Amplifiers and Buffers"
- note added: "Power"
- note added: "Spare"
- note added: "Used"
- note removed: "CV Input Scaling"
- note removed: "Power Sections"
- note removed: "Use PA4 and PA5 which\n we need for DAC"
- moved on the sheet: C1, C10, C11, C12, C13, C14, C15, C16, C17, C18, C19, C2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

Commit message: Initial pass at routing MCU and DRAM
Parts:
- U2: footprint Package_SO:TSOP-II-54_10.16x22.22mm_P0.8mm -> Custom_Footprints:TSOP-II-54_22.2x10.16mm_P0.8mm
- U4: footprint Package_SO:SOIC-16_3.9x9.9mm_P1.27mm -> Housings_SOIC:SOIC-16_3.9x9.9mm_Pitch1.27mm
Connections:
- net ADC12_INP14_PA2_IN is gone; now on net ADC12_INP14_PA2: J5.6 (Pin_6)
- net ADC12_INP7 is gone; now on net FEEDBACK_CV_SCALED: U1.43 (PA7)
- net ADC12_INP7_PA7_IN is gone; now on net ADC12_INP7_PA7: J5.5 (Pin_5)
- net ADC12_INP9 is gone; now on net FEEDBACK_POT: U1.46 (PB0)
- net AUDIO_L is gone; now on net AUDIO_IN_L: R1.2
- net AUDIO_R is gone; now on net AUDIO_IN_R: R2.2
- net +3.3VA: now also C21.2; no longer C11.2
- net +3V3: now also C11.2; no longer C21.2
- net AUDIO_IN_L: now also U1.42 (PA6)
- net AUDIO_IN_R: now also U1.27 (PC1)
- net DELAY_CV_L: no longer U1.44 (PC4)
- net DELAY_CV_SCALED_R: now also U1.44 (PC4)
- net EXT_AUDIO_IN_L: no longer U1.42 (PA6)
- net EXT_AUDIO_IN_R: no longer U1.27 (PC1)
- net LED1: now also U1.111 (PC10)
- net LED2: now also U1.112 (PC11)
- net MODE1: now also U1.97 (PC7)
- net MODE2: now also U1.98 (PC8)
- net ADC12_INP14: no longer names the net of U1.36 (PA2)
- no-connect marks 71 -> 68
Other:
- moved on the sheet: C1, C10, C11, C21, C36, C38, C39, C40, C41, C43, C45, C5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
