File: Hardware/_autosave-Alligator_Components.kicad_pcb (KiCad board)
At the start: 4 copper layers, 60 x 110 mm, 114 parts, among them J1 SWD_Header, J2 Eurorack_10_pin_power, J3 Conn_01x08_Female, J4 Conn_01x08_Female, J5 Conn_01x08_Female, J6 Conn_01x08_Female, SW1 SW_SPST, SW2 SW_SPDT_MSM, U1 STM32H743ZITx, U2 IS42S16400J-xC, U3 PCM5100APW, U4 SSI2164, U5 MCP6004, U6 MCP6004, U7 TL074, U8 LM1117-3.3, Y1 8MHz 20pF

Commit message: Continued routing and reorganising PCB
Routing:
- net /DRY_OUT_R: track 4.66 -> 10.1 mm
- net /DRY_OUT_L: track 4.66 -> 10.1 mm
Changed lines of the file:
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@@
     (thickness 1.6)
     (drawings 4)
-    (tracks 775)
+    (tracks 779)
     (zones 0)
     (modules 114)
@@
   (segment (start 138.54 78.24) (end 138.1 77.8) (width 0.25) (layer F.Cu) (net 45) (status 30))
   (segment (start 138.54 79.952) (end 138.54 78.24) (width 0.25) (layer F.Cu) (net 45) (status 30))
+  (segment (start 115.265 71.3) (end 115.265 75.7) (width 0.25) (layer F.Cu) (net 45))
+  (segment (start 115.265 70.3) (end 115.265 71.3) (width 0.25) (layer F.Cu) (net 45))
   (segment (start 131.7 79.462) (end 132.19 79.952) (width 0.25) (layer F.Cu) (net 46) (status 20))
   (segment (start 131.7 77.8) (end 131.7 79.462) (width 0.25) (layer F.Cu) (net 46) (status 10))
@@
   (segment (start 133.46 78.24) (end 133.9 77.8) (width 0.25) (layer F.Cu) (net 47) (status 30))
   (segment (start 133.46 79.952) (end 133.46 78.24) (width 0.25) (layer F.Cu) (net 47) (status 30))
+  (segment (start 116.535 71.3) (end 116.535 75.7) (width 0.25) (layer F.Cu) (net 47))
+  (segment (start 116.535 70.3) (end 116.535 71.3) (width 0.25) (layer F.Cu) (net 47))
   (segment (start 141.849999 134.385001) (end 141.914999 134.450001) (width 0.25) (layer F.Cu) (net 48))
   (segment (start 141.849999 130.864999) (end 141.849999 134.385001) (width 0.25) (layer F.Cu) (net 48))
