File: Hardware/Retrospector_Power_Test_LM2675.sch (KiCad schematic (older format))
At the start: 21 parts, among them J2 Eurorack_10_pin_power, U1 LM2675M-ADJ, U2 LD1117-3.3-4Tab

Commit message: Added project to support STM32F429 using same hardware; all components tested and working except I2S DAC
Other:
- note added: "3.3V\n\n1.74k\n1k\n47uH\n22uF+100nF\n100uF\n\n969uV\n260kHz"
- note added: "5V\n\n10k\n3.24k\n68uH\n10uF\n100uF\n\n9mV\n500kHz"
- note added: "5V\n\n3.16k\n1k\n68uF\n22uF+100nF\n47uF\n\n13mV\n260kHz"
- note added: "Input Capacitor\nCeramic, XR5 1210"
- note added: "NB - no good as output capacitor too large"
- note removed: "3.3V\n\n1.74k\n1k\n47uH\n33uF+100nF\n100uF\n\n15.5mV\n260kHz"
- note removed: "5V\n\n10k\n3.24k\n68uH\n10uF\n100uF"
- note removed: "5V\n\n3.16k\n1k\n68uF\n100uF+100nF\n47uF\n\n13mV\n260kHz"
- note removed: "Input Capacitor\nCeramic, XR5 1206"
Changed lines of the file:
@@
 For 5V output change:\n- Output Capacitor from 150uF to 100uF\n- Lower FB resistor from 5.9k to 3.24k\nNB 5.6k gives output of 3.4V; 6.2k gives 3.2V
 Text Notes 550  3650 0    50   ~ 0
-Input Capacitor\nCeramic, XR5 1206
+Input Capacitor\nCeramic, XR5 1210
 $Comp
 L Device:C_Small C2
@@
 Text Notes 6000 1000 0    50   ~ 0
 LM2675
-Text Notes 7050 1000 0    50   ~ 0
+Text Notes 7600 1000 0    50   ~ 0
 TPS5410
 Text Notes 5750 1900 0    50   ~ 0
-3.3V\n\n1.74k\n1k\n47uH\n33uF+100nF\n100uF\n\n15.5mV\n260kHz
+3.3V\n\n1.74k\n1k\n47uH\n22uF+100nF\n100uF\n\n969uV\n260kHz
 Text Notes 6300 1900 0    50   ~ 0
-5V\n\n3.16k\n1k\n68uF\n100uF+100nF\n47uF\n\n13mV\n260kHz
-Text Notes 6900 1900 0    50   ~ 0
+5V\n\n3.16k\n1k\n68uF\n22uF+100nF\n47uF\n\n13mV\n260kHz
+Text Notes 8000 1900 0    50   ~ 0
+5V\n\n10k\n3.24k\n68uH\n10uF\n100uF\n\n9mV\n500kHz
+Text Notes 7450 1900 0    50   ~ 0
 3.3V\n\n10k\n5.9k\n68uH\n10uF\n150uF\n\n6.2mV\n500kHz
-Text Notes 7450 1650 0    50   ~ 0
-5V\n\n10k\n3.24k\n68uH\n10uF\n100uF
+Text Notes 7200 2100 0    50   ~ 0
+NB - no good as output capacitor too large
 $EndSCHEMATC

Commit message: Debugging DAC clock issues when using FMC to control SDRAM
Workaround is to switch the clock for the I2S DAC to peripheral clock (also used by ADC at present)
Parts:
- C2: value 10uF -> 22uF
- C4: value 150uF -> 100uF
- R1: value 1.74k -> 1k8
Changed lines of the file:
@@
 P 4000 3350
 F 0 "C4" H 4088 3396 50  0000 L CNN
-F 1 "150uF" H 4088 3305 50  0000 L CNN
+F 1 "100uF" H 4088 3305 50  0000 L CNN
 F 2 "Capacitors_SMD:C_1210" H 4000 3350 50  0001 C CNN
 F 3 "https://datasheet.lcsc.com/szlcsc/1809131544_PANASONIC-EEEFT1V220AR_C178597.pdf" H 4000 3350 50  0001 C CNN
@@
 P 3550 3150
 F 0 "R1" H 3609 3196 50  0000 L CNN
-F 1 "1.74k" H 3609 3105 50  0000 L CNN
+F 1 "1k8" H 3609 3105 50  0000 L CNN
 F 2 "Resistors_SMD:R_0603_HandSoldering" H 3550 3150 50  0001 C CNN
 F 3 "~" H 3550 3150 50  0001 C CNN
@@
 P 1300 3300
 F 0 "C2" H 1150 3300 50  0000 C CNN
-F 1 "10uF" H 1200 3200 50  0000 C CNN
+F 1 "22uF" H 1200 3200 50  0000 C CNN
 F 2 "Capacitors_SMD:C_1210" H 1300 3300 50  0001 C CNN
 F 3 "~" H 1300 3300 50  0001 C CNN

Commit message: More clock experiments
Other:
- note added: "5V\n\n3.16k\n1k\n68uH\n22uF+100nF\n47uF\n\n13mV\n260kHz"
- note removed: "5V\n\n3.16k\n1k\n68uF\n22uF+100nF\n47uF\n\n13mV\n260kHz"
Changed lines of the file:
@@
 3.3V\n\n1.74k\n1k\n47uH\n22uF+100nF\n100uF\n\n969uV\n260kHz
 Text Notes 6300 1900 0    50   ~ 0
-5V\n\n3.16k\n1k\n68uF\n22uF+100nF\n47uF\n\n13mV\n260kHz
+5V\n\n3.16k\n1k\n68uH\n22uF+100nF\n47uF\n\n13mV\n260kHz
 Text Notes 8000 1900 0    50   ~ 0
 5V\n\n10k\n3.24k\n68uH\n10uF\n100uF\n\n9mV\n500kHz
