File: Hardware/Retrospector_Controls.sch (KiCad schematic (older format))
At the start: 32 parts, among them J1 Conn_01x08_Female, J10 Feedback_CV, J11 Audio_In_R, J12 Audio_Out_R, J13 Audio_Out_L, J14 Filter, J2 Conn_01x08_Female, J3 Conn_01x08_Female, J4 Conn_01x08_Female, J5 Audio_In_L, J6 Delay_CV_L, J7 Mix_CV, J8 Delay_CV_R, J9 Clock, U1 TB62781FNG

Commit message: Final updates to v2 PCBs for production; USB DFU Mode working
Changed lines of the file:
@@
 Text Label 3100 2000 0    50   ~ 0
 DELAY_CV_R
-Text Label 4600 1100 0    50   ~ 0
+Text Label 4650 1100 0    50   ~ 0
 FEEDBACK_CV
 Text Label 4650 2000 0    50   ~ 0
@@
 L thonkiconn:AudioJack2_Ground_Switch J10
 U 1 1 5F88B48E
-P 4200 1100
-F 0 "J10" H 4205 1442 50  0000 C CNN
-F 1 "Feedback_CV" H 4205 1351 50  0000 C CNN
-F 2 "Custom_Footprints:THONKICONN_hole" H 4200 1100 50  0001 C CNN
-F 3 "~" H 4200 1100 50  0001 C CNN
-	1    4200 1100
+P 4250 1100
+F 0 "J10" H 4255 1442 50  0000 C CNN
+F 1 "Feedback_CV" H 4255 1351 50  0000 C CNN
+F 2 "Custom_Footprints:THONKICONN_hole" H 4250 1100 50  0001 C CNN
+F 3 "~" H 4250 1100 50  0001 C CNN
+	1    4250 1100
 	1    0    0    -1
 $EndComp
@@
 L power:GND #PWR05
 U 1 1 5F88B494
-P 4500 1300
-F 0 "#PWR05" H 4500 1050 50  0001 C CNN
-F 1 "GND" H 4505 1127 50  0000 C CNN
-F 2 "" H 4500 1300 50  0001 C CNN
-F 3 "" H 4500 1300 50  0001 C CNN
-	1    4500 1300
-	1    0    0    -1
-$EndComp
-Wire Wire Line
-	4400 1000 4500 1000
-Wire Wire Line
-	4500 1000 4500 1200
-Wire Wire Line
-	4400 1100 4600 1100
-Wire Wire Line
-	4400 1200 4500 1200
-Connection ~ 4500 1200
-Wire Wire Line
-	4500 1200 4500 1300
+P 4550 1300
+F 0 "#PWR05" H 4550 1050 50  0001 C CNN
+F 1 "GND" H 4555 1127 50  0000 C CNN
+F 2 "" H 4550 1300 50  0001 C CNN
+F 3 "" H 4550 1300 50  0001 C CNN
+	1    4550 1300
+	1    0    0    -1
+$EndComp
+Wire Wire Line
+	4450 1000 4550 1000
+Wire Wire Line
+	4550 1000 4550 1200
+Wire Wire Line
+	4450 1100 4650 1100
+Wire Wire Line
+	4450 1200 4550 1200
+Connection ~ 4550 1200
+Wire Wire Line
+	4550 1200 4550 1300
 Text Label 3100 1100 0    50   ~ 0
 DELAY_CV_L
@@
 $EndComp
 Wire Wire Line
-	6100 4100 5950 4100
-Wire Wire Line
-	5950 4100 5950 4600
-Wire Wire Line
-	5950 4600 5400 4600
-Wire Wire Line
-	6100 4300 6000 4300
-Wire Wire Line
-	6000 4300 6000 4700
-Wire Wire Line
-	6000 4700 5400 4700
-Wire Wire Line
-	6100 4500 6050 4500
-Wire Wire Line
-	6050 4500 6050 4800
-Wire Wire Line
-	6050 4800 5400 4800
+	6100 4100 5900 4100
+Wire Wire Line
+	5900 4100 5900 4600
+Wire Wire Line
+	5900 4600 5400 4600
+Wire Wire Line
+	6100 4300 5950 4300
+Wire Wire Line
+	5950 4300 5950 4700
+Wire Wire Line
+	5950 4700 5400 4700
+Wire Wire Line
+	6100 4500 6000 4500
+Wire Wire Line
+	6000 4500 6000 4800
+Wire Wire Line
+	6000 4800 5400 4800
 Wire Wire Line
 	6100 5000 6050 5000

Commit message: Corrections to PCB for v3; implemented filter mode switch
Connections:
- net labels added: STEREO_WIDE
- net labels removed: PINGPONG
Changed lines of the file:
@@
 MODE2
 Text Label 2300 5550 0    50   ~ 0
-CHORUS
+STEREO_WIDE
 Text Label 2300 4200 0    50   ~ 0
 MODE1
@@
 Headers
 Text Label 2300 5450 0    50   ~ 0
-PINGPONG
+CHORUS
 Text Label 2300 5350 0    50   ~ 0
 LINK_BTN
@@
 $EndComp
 Text Label 8050 1900 2    50   ~ 0
+STEREO_WIDE
+Text Label 8050 2100 2    50   ~ 0
 CHORUS
-Text Label 8050 2100 2    50   ~ 0
-PINGPONG
 $Comp
 L power:PWR_FLAG #FLG0103

Commit message: Tests with filter led
Parts:
- R1, R2, R3: value 3k3 -> 10k
Changed lines of the file:
@@
 P 4150 5200
 F 0 "R1" V 4100 5050 50  0000 C CNN
-F 1 "3k3" V 4150 5200 30  0000 C CNN
+F 1 "10k" V 4150 5200 30  0000 C CNN
 F 2 "Resistors_SMD:R_0603_HandSoldering" H 4150 5200 50  0001 C CNN
 F 3 "~" H 4150 5200 50  0001 C CNN
@@
 P 4150 5300
 F 0 "R2" V 4100 5150 50  0000 C CNN
-F 1 "3k3" V 4150 5300 30  0000 C CNN
+F 1 "10k" V 4150 5300 30  0000 C CNN
 F 2 "Resistors_SMD:R_0603_HandSoldering" H 4150 5300 50  0001 C CNN
 F 3 "~" H 4150 5300 50  0001 C CNN
@@
 P 4150 5400
 F 0 "R3" V 4100 5250 50  0000 C CNN
-F 1 "3k3" V 4150 5400 30  0000 C CNN
+F 1 "10k" V 4150 5400 30  0000 C CNN
 F 2 "Resistors_SMD:R_0603_HandSoldering" H 4150 5400 50  0001 C CNN
 F 3 "~" H 4150 5400 50  0001 C CNN
