File: Hardware/Retrospector_Components.kicad_sch (KiCad schematic)
At the start: 149 parts, among them J1 Conn_01x08_Male, J2 Conn_01x08_Male, J3 Conn_01x08_Male, J4 Conn_01x08_Male, J5 SWD_Header, J6 USB_B_Micro, J7 Eurorack_10_pin_power, J8 I2C_TestPoint, U1 MCP6004, U10 LD1117-3.3-4Tab, U2 TL074, U3 MCP6004, U4 IS42S16800F-7TLI, U5 STM32H743ZITx, U6 TL072, U7 AS3364, U8 PCM5100APW, U9 LM2675M-5, Y1 8MHz 20pF

Commit message: Cleaned up hardware folder
Parts:
- removed U?: Hyperram_BGA, symbol Hyperram:Hyperram_BGA
Connections:
- net FMC_A6: no longer U4.17 (~{CAS}), U5.132 (PG15)
- new net FMC_~{CAS}: U4.17 (~{CAS}), U5.132 (PG15)
