File: Hardware_v2/Retrospector_Components.sch (KiCad schematic (older format))
At the start: 145 parts, among them J1 SWD_Header, J2 Eurorack_10_pin_power, J3 Conn_01x08_Male, J4 Conn_01x08_Male, J5 Conn_01x08_Male, J6 Conn_01x08_Male, J7 USB_B_Micro, U1 STM32H743ZITx, U10 LM2675M-5, U11 TL072, U2 IS42S16800F-7TLI, U3 PCM5100APW, U4 SSI2164, U5 MCP6004, U6 MCP6004, U7 TL074, U8 LD1117-3.3-4Tab, Y1 8MHz 20pF

Commit message: Started work on v3 of PCB layout and schematic
Parts:
- removed R45, R46, R47, R48: 10k, Resistors_SMD:R_0603_HandSoldering, symbol Device:R
- removed TP10, TP11, TP12: TestPoint, Measurement_Points:Measurement_Point_Square-SMD-Pad_Small, symbol Connector:TestPoint
- removed U8: LD1117-3.3-4Tab, TO_SOT_Packages_SMD:SOT-223-3_TabPin2, symbol LD1117-3.3-4Tab:LD1117-3.3-4Tab
- added U8: NCV1117DT33T5G, TO_SOT_Packages_SMD:TO-252-2_Rectifier, symbol LDO_DPAK:NCV1117DT33T5G
- J7: symbol Connector:USB_B_Micro -> Retrospector_Components-rescue:USB_B_Micro-Connector
Connections:
- wire segments 647 -> 643
- no-connect marks 47 -> 49
Other:
- moved on the sheet: R20, R21, TP1, TP2, TP3, TP4, TP5, TP6, TP7, TP8, TP9, U11A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
